File: TXB0108DQSR-breakout/TXB0108DQSR-breakout.kicad_pcb (KiCad board)
At the start: 2 copper layers, 13.7 x 26.4 mm, 8 parts, among them J1 Conn_01x10_Male, J2 Conn_01x10_Male, U1 TXB0108DQSR

Commit message: update kicad_pcb ver 0.1
Other:
- board text added: "Ver 0.1"
Changed lines of the file:
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@@
   (general
     (thickness 1.6)
-    (drawings 28)
+    (drawings 29)
     (tracks 105)
     (zones 0)
@@
     )
   )
+  (gr_text "Ver 0.1" (at 147.447 96.4946 180) (layer B.SilkS)
+    (effects (font (size 0.75 0.75) (thickness 0.15)) (justify mirror))
+  )
   (gr_text "NOV 2020" (at 147.2946 74.6252 180) (layer B.SilkS)
